File: simulation/PCBDesign1/PCBDesign1.kicad_sch (KiCad schematic)
At the start: 77 parts, among them J2 Conn_02x16_Counter_Clockwise, J3 Conn_01x02, J4 TYPE-C-31-M-12, Q1 2N7002, U1 CH224K, U10 TPS2553DBVR, U11 TPS2553DBVR, U2 BQ24074RGT, U3 TPS62200DBV, U4 MT3608, U5 DRV8835DSSR, U6 DRV8835DSSR, U7 INA219AxDCN

Commit message: Restructured repo: keep README at root and add simulation/pcbdesign1
Other:
- note added: "This asks from the USB-C for 9V and is done so through the configuration of 000 for the CFG pins VBUS then provides this out to the Battery Charger circuit below. The various pins connected between are for communication (CC1-2, DM, DP)."
- note added: "This is now the hub between the USB-C, the battery and the rest of the circuit. Notes: - EN1, EN2 set to high current mode, outputs 1.5A (logic 1,1) - ISET controls charge current (Iset = 890/R4) need 600mA or 200mA - RITERM = (ITERM * RISET)/0.03, had to choose between 2.2k-3k - FLoating: TMR - CHG = 0 when charging and PGOOD = 0 when power good, else floating"
- note added: "This is purely the USB-C connection with shield as protection. It connects to the CHK224K for the negotiation. The USB-C is setup in a way to only provide power and not the transfer of data. It has been configured this way."
- note added: "This is the high-side switch with some proection Notes:-IN is connected to the 5V rail and OUT powers the load. - EN is active-high and controlled by logic from stm - ILIM limits the current. Ilim = 1350/RIlim"
- note removed: "- EN1, EN2 set to high current mode, outputs 1.5A (gets logic 1,1) - ISET controls charge current (Iset = 890/R4) need 600mA or 200mA - RITERM = (ITERM * RISET)/0.03, had to choose between 2.2k-3k - FLoating: TMR - CHG = 0 when charging and PGOOD = 0 when power good, else floating"
- note removed: "Notes: Configure 000 for the CFG's to negotiate for the 9V. VBUS provides the 9V."
- note removed: "Shield is just protection. It can go to ground or the setup we have"
- company: (none) -> University Of Cape Town
- title: (none) -> Power Subsystem Design V7
- moved on the sheet: C10, C11, C12, C13, C14, C17, C18, C2, C3, C4, C5, C6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
